Commit message: chore: snapshot current A1Z workspace

File: build/robot_packages/A1Z_G1Z/urdf/A1Z_G1Z.urdf (robot description, URDF)
Before this commit: robot A1Z_G1Z, 9 links, 8 joints
Joints:
- joint arm_joint1: limit lower=-2.094 upper=2.094 effort=0 velocity=0 -> lower=-2.094 upper=2.094 effort=20 velocity=5.65
- joint arm_joint2: limit lower=0 upper=3.142 effort=0 velocity=0 -> lower=0 upper=3.142 effort=25 velocity=5.65
- joint arm_joint3: limit lower=-3.142 upper=0 effort=0 velocity=0 -> lower=-3.142 upper=0 effort=20 velocity=5.65
- joint arm_joint4: limit lower=-1.309 upper=1.309 effort=0 velocity=0 -> lower=-1.309 upper=1.309 effort=9 velocity=3.77
- joint arm_joint5: limit lower=-1.484 upper=1.484 effort=0 velocity=0 -> lower=-1.484 upper=1.484 effort=3.5 velocity=10.47
- joint arm_joint6: limit lower=-2.007 upper=2.007 effort=0 velocity=0 -> lower=-2.007 upper=2.007 effort=3.5 velocity=10.47
- joint gripper_finger_left_joint: axis 0 1 0 -> (none); limit lower=0 upper=0.048 effort=0 velocity=0 -> (none); type prismatic -> fixed
- joint gripper_finger_rIght_joint: axis 0 1 0 -> (none); limit lower=-0.048 upper=0 effort=0 velocity=0 -> (none); mimic joint=gripper_finger_left_joint multiplier=-1 offset=0 -> (none); type prismatic -> fixed

File: build/robot_packages/A1Z_G1Z/urdf/A1Z_G1Z_control.urdf (robot description, URDF)
Before this commit: robot A1Z_G1Z, 10 links, 9 joints
Links:
- link d405_link: mass 0.072 -> 0.001
Joints:
- joint arm_joint1: limit lower=-2.094 upper=2.094 effort=20 velocity=5.65 -> lower=-2.094395 upper=2.094395 effort=20 velocity=5.654867
- joint arm_joint2: limit lower=0 upper=3.142 effort=25 velocity=5.65 -> lower=0 upper=3.141593 effort=25 velocity=5.654867
- joint arm_joint3: limit lower=-3.142 upper=0 effort=20 velocity=5.65 -> lower=-3.141593 upper=0 effort=20 velocity=5.654867
- joint arm_joint4: limit lower=-1.309 upper=1.309 effort=9 velocity=3.77 -> lower=-1.48353 upper=1.48353 effort=9 velocity=3.769911
- joint arm_joint5: limit lower=-1.484 upper=1.484 effort=3.5 velocity=10.47 -> lower=-1.48353 upper=1.48353 effort=3.5 velocity=10.471976
- joint arm_joint6: limit lower=-2.007 upper=2.007 effort=3.5 velocity=10.47 -> lower=-2.007129 upper=2.007129 effort=3.5 velocity=10.471976
- joint d405_mount_joint: origin xyz=0.09238 0 0.09625 rpy=2.2724490548256018 0 1.5707963267948966 -> xyz=0.08 0 0.086237 rpy=2.251475 0 1.570796

File: build/robot_packages/A1Z_G1Z/urdf/A1Z_G1Z_isaac.urdf (robot description, URDF)
Before this commit: robot A1Z_G1Z, 10 links, 9 joints
Links:
- link d405_link: mass 0.072 -> 0.001
Joints:
- joint arm_joint1: limit lower=-2.094 upper=2.094 effort=0 velocity=0 -> lower=-2.268928 upper=2.268928 effort=20 velocity=5.654867
- joint arm_joint2: limit lower=0 upper=3.142 effort=0 velocity=0 -> lower=-0.033859 upper=3.364646 effort=25 velocity=5.654867
- joint arm_joint3: limit lower=-3.142 upper=0 effort=0 velocity=0 -> lower=-3.497291 upper=0 effort=20 velocity=5.654867
- joint arm_joint4: limit lower=-1.309 upper=1.309 effort=0 velocity=0 -> lower=-1.603609 upper=1.926494 effort=9 velocity=3.769911
- joint arm_joint5: limit lower=-1.484 upper=1.484 effort=0 velocity=0 -> lower=-1.570796 upper=1.570796 effort=3.5 velocity=10.471976
- joint arm_joint6: limit lower=-2.007 upper=2.007 effort=0 velocity=0 -> lower=-2.094395 upper=2.094395 effort=3.5 velocity=10.471976
- joint d405_mount_joint: origin xyz=0.09238 0 0.09625 rpy=2.2724490548256018 0 1.5707963267948966 -> xyz=0.08 0 0.086237 rpy=2.251475 0 1.570796
- joint gripper_finger_left_joint: axis 0 1 0 -> (none); limit lower=0 upper=0.048 effort=0 velocity=0 -> (none)
- joint gripper_finger_rIght_joint: axis 0 1 0 -> (none); limit lower=-0.048 upper=0 effort=0 velocity=0 -> (none); mimic joint=gripper_finger_left_joint multiplier=-1 offset=0 -> (none)

File: vendor/GALAXEA-A1Z/a1z/robot_models/a1z/A1Z_G1Z.urdf (robot description, URDF)
Before this commit: robot A1Z_G1Z, 10 links, 9 joints
Links:
- removed link d405_link
Joints:
- removed joint d405_mount_joint
- joint arm_joint1: limit lower=-2.094 upper=2.094 effort=0 velocity=0 -> lower=-2.094 upper=2.094 effort=20 velocity=5.65
- joint arm_joint2: limit lower=0 upper=3.142 effort=0 velocity=0 -> lower=0 upper=3.142 effort=25 velocity=5.65
- joint arm_joint3: limit lower=-3.142 upper=0 effort=0 velocity=0 -> lower=-3.142 upper=0 effort=20 velocity=5.65
- joint arm_joint4: limit lower=-1.309 upper=1.309 effort=0 velocity=0 -> lower=-1.309 upper=1.309 effort=9 velocity=3.77
- joint arm_joint5: limit lower=-1.484 upper=1.484 effort=0 velocity=0 -> lower=-1.484 upper=1.484 effort=3.5 velocity=10.47
- joint arm_joint6: limit lower=-2.007 upper=2.007 effort=0 velocity=0 -> lower=-2.007 upper=2.007 effort=3.5 velocity=10.47
- joint gripper_finger_left_joint: axis 0 1 0 -> (none); limit lower=0 upper=0.048 effort=0 velocity=0 -> (none); type prismatic -> fixed
- joint gripper_finger_rIght_joint: axis 0 1 0 -> (none); limit lower=-0.048 upper=0 effort=0 velocity=0 -> (none); mimic joint=gripper_finger_left_joint multiplier=-1 offset=0 -> (none); type prismatic -> fixed
