Commit message: feat: add perception and grasping pipeline tooling

File: build/robot_packages/A1Z_G1Z/urdf/A1Z_G1Z_isaac.urdf (robot description, URDF)
Before this commit: robot A1Z_G1Z, 10 links, 9 joints
Joints:
- joint gripper_finger_left_joint: axis (none) -> 0 1 0
- joint gripper_finger_rIght_joint: axis (none) -> 0 1 0
