Commit message: Update vision tooling and rebuild generated assets

File: build/robot_packages/A1Z_G1Z/urdf/A1Z_G1Z_control.urdf (robot description, URDF)
Before this commit: robot A1Z_G1Z, 10 links, 9 joints
Joints:
- joint d405_mount_joint: origin xyz=0.08 0 0.086237 rpy=2.251475 0 1.570796 -> xyz=0 0 0.056237 rpy=0 0 0

File: build/robot_packages/A1Z_G1Z/urdf/A1Z_G1Z_isaac.urdf (robot description, URDF)
Before this commit: robot A1Z_G1Z, 10 links, 9 joints
Joints:
- joint d405_mount_joint: origin xyz=0.08 0 0.086237 rpy=2.251475 0 1.570796 -> xyz=0 0 0.056237 rpy=0 0 0
