Commit message: Integrate Isaac grasping and tooling updates

File: build/robot_packages/A1Z_G1Z/urdf/A1Z_G1Z_control.urdf (robot description, URDF)
Before this commit: robot A1Z_G1Z, 10 links, 9 joints
Links:
- link arm_link3: mass 0.99109270 -> 0.939545
- link arm_link4: mass 0.48309874 -> 0.177099
- link arm_link5: mass 0.36875049 -> 0.36875
- link arm_link6: mass 0.55665538 -> 0.423356
- link d405_link: geometry visual mesh filename=package://A1Z_G1Z/meshes/d405.stl scale=0.001 0.001 0.001
Joints:
- joint d405_mount_joint: origin xyz=0 0 0.056237 rpy=0 0 0 -> xyz=0.08 0 0.086237 rpy=2.251475 0 1.570796

File: build/robot_packages/A1Z_G1Z/urdf/A1Z_G1Z_isaac.urdf (robot description, URDF)
Before this commit: robot A1Z_G1Z, 10 links, 9 joints
Links:
- link arm_link3: mass 0.99109270 -> 0.939545
- link arm_link4: mass 0.48309874 -> 0.177099
- link arm_link5: mass 0.36875049 -> 0.36875
- link arm_link6: mass 0.55665538 -> 0.423356
- link d405_link: geometry visual mesh filename=package://A1Z_G1Z/meshes/d405.stl scale=0.001 0.001 0.001
Joints:
- joint d405_mount_joint: origin xyz=0 0 0.056237 rpy=0 0 0 -> xyz=0.08 0 0.086237 rpy=2.251475 0 1.570796

Commit message: Update AnyGrasp, D405 frame chain, and motion TF config

File: build/robot_packages/A1Z_G1Z/urdf/A1Z_G1Z_control.urdf (robot description, URDF)
Before this commit: robot A1Z_G1Z, 10 links, 9 joints
Links:
- added link d405_rectified_link
- added link grasp_tcp
Joints:
- added joint d405_rectified_joint: type fixed, parent d405_link, child d405_rectified_link, origin xyz=0 0 0 rpy=0 0 0
- added joint grasp_tcp_joint: type fixed, parent arm_link6, child grasp_tcp, origin xyz=0.04 0 0 rpy=0 0 0
- joint d405_mount_joint: origin xyz=0.08 0 0.086237 rpy=2.251475 0 1.570796 -> xyz=0.08 0 0.086237 rpy=0 0 0

File: build/robot_packages/A1Z_G1Z/urdf/A1Z_G1Z_isaac.urdf (robot description, URDF)
Before this commit: robot A1Z_G1Z, 10 links, 9 joints
Links:
- added link d405_rectified_link
- added link grasp_tcp
Joints:
- added joint d405_rectified_joint: type fixed, parent d405_link, child d405_rectified_link, origin xyz=0 0 0 rpy=0 0 0
- added joint grasp_tcp_joint: type fixed, parent arm_link6, child grasp_tcp, origin xyz=0.04 0 0 rpy=0 0 0
- joint d405_mount_joint: origin xyz=0.08 0 0.086237 rpy=2.251475 0 1.570796 -> xyz=0.08 0 0.086237 rpy=0 0 0

Commit message: Align AnyGrasp TCP defaults with approach-x mapping

File: build/robot_packages/A1Z_G1Z/urdf/A1Z_G1Z_control.urdf (robot description, URDF)
Before this commit: robot A1Z_G1Z, 12 links, 11 joints
Joints:
- joint grasp_tcp_joint: origin xyz=0.04 0 0 rpy=0 0 0 -> xyz=0.08 0 0 rpy=0 0 0

File: build/robot_packages/A1Z_G1Z/urdf/A1Z_G1Z_isaac.urdf (robot description, URDF)
Before this commit: robot A1Z_G1Z, 12 links, 11 joints
Joints:
- joint grasp_tcp_joint: origin xyz=0.04 0 0 rpy=0 0 0 -> xyz=0.08 0 0 rpy=0 0 0

Commit message: feat: complete Isaac 6 force closed-loop migration

File: build/robot_packages/A1Z_G1Z/urdf/A1Z_G1Z_control.urdf (robot description, URDF)
Before this commit: robot A1Z_G1Z, 12 links, 11 joints
Links:
- link gripper_finger_left_link: mass 0.13786800 -> 0.02
- link gripper_finger_rIght_link: mass 0.13786800 -> 0.02

File: build/robot_packages/A1Z_G1Z/urdf/A1Z_G1Z_isaac.urdf (robot description, URDF)
Before this commit: robot A1Z_G1Z, 12 links, 11 joints
Links:
- link gripper_finger_left_link: mass 0.13786800 -> 0.02
- link gripper_finger_rIght_link: mass 0.13786800 -> 0.02
Joints:
- joint gripper_finger_left_joint: limit (none) -> lower=0 upper=0.048 effort=120 velocity=0.35
- joint gripper_finger_rIght_joint: limit (none) -> lower=-0.048 upper=0 effort=120 velocity=0.35

Commit message: feat: add A1Z SDK console and D405 integration

File: build/robot_packages/A1Z_G1Z/urdf/A1Z_G1Z_control.urdf (robot description, URDF)
Before this commit: robot A1Z_G1Z, 12 links, 11 joints
Links:
- added link camera_bracket_link, mass 0.03; visual mesh filename=package://A1Z_G1Z/meshes/camera_bracket.stl scale=0.001 0.001 0.001
Joints:
- added joint camera_bracket_mount_joint: type fixed, parent arm_link6, child camera_bracket_link, origin xyz=0.06842 0 0.06546 rpy=-1.57079632679 0 1.57079632679
- joint d405_mount_joint: origin xyz=0.08 0 0.086237 rpy=0 0 0 -> xyz=0.0650543901297 0 0.0837692743183 rpy=0 -0.181432196149 0

File: build/robot_packages/A1Z_G1Z/urdf/A1Z_G1Z_isaac.urdf (robot description, URDF)
Before this commit: robot A1Z_G1Z, 12 links, 11 joints
Links:
- added link camera_bracket_link, mass 0.03; visual mesh filename=package://A1Z_G1Z/meshes/camera_bracket.stl scale=0.001 0.001 0.001
Joints:
- added joint camera_bracket_mount_joint: type fixed, parent arm_link6, child camera_bracket_link, origin xyz=0.06842 0 0.06546 rpy=-1.57079632679 0 1.57079632679
- joint d405_mount_joint: origin xyz=0.08 0 0.086237 rpy=0 0 0 -> xyz=0.0650543901297 0 0.0837692743183 rpy=0 -0.181432196149 0

Commit message: Restore payload dynamics and improve console controls

File: build/robot_packages/A1Z_G1Z/urdf/A1Z_G1Z_control.urdf (robot description, URDF)
Before this commit: robot A1Z_G1Z, 13 links, 12 joints
Links:
- link arm_link3: mass 0.939545 -> 0.99109270
- link arm_link4: mass 0.177099 -> 0.48309874
- link arm_link5: mass 0.36875 -> 0.36875049
- link arm_link6: mass 0.423356 -> 0.55665538
- link d405_link: mass 0.001 -> 0.072
- link gripper_finger_left_link: mass 0.02 -> 0.13786800
- link gripper_finger_rIght_link: mass 0.02 -> 0.13786800

File: build/robot_packages/A1Z_G1Z/urdf/A1Z_G1Z_isaac.urdf (robot description, URDF)
Before this commit: robot A1Z_G1Z, 13 links, 12 joints
Links:
- link arm_link3: mass 0.939545 -> 0.99109270
- link arm_link4: mass 0.177099 -> 0.48309874
- link arm_link5: mass 0.36875 -> 0.36875049
- link arm_link6: mass 0.423356 -> 0.55665538
- link d405_link: mass 0.001 -> 0.072
- link gripper_finger_left_link: mass 0.02 -> 0.13786800
- link gripper_finger_rIght_link: mass 0.02 -> 0.13786800

Commit message: Fix A1Z link6 inertia and gravity validation

File: build/robot_packages/A1Z_G1Z/urdf/A1Z_G1Z_control.urdf (robot description, URDF)
Before this commit: robot A1Z_G1Z, 13 links, 12 joints
Links:
- link arm_link6: mass 0.55665538 -> 0.42335647

File: build/robot_packages/A1Z_G1Z/urdf/A1Z_G1Z_isaac.urdf (robot description, URDF)
Before this commit: robot A1Z_G1Z, 13 links, 12 joints
Links:
- link arm_link6: mass 0.55665538 -> 0.42335647

Commit message: refine sth

File: build/robot_packages/A1Z_G1Z/urdf/A1Z_G1Z_control.urdf (robot description, URDF)
Before this commit: robot A1Z_G1Z, 13 links, 12 joints
Links:
- link camera_bracket_link: mass 0.03 -> 0.0292706516842
- link d405_link: mass 0.072 -> 0.06

File: build/robot_packages/A1Z_G1Z/urdf/A1Z_G1Z_isaac.urdf (robot description, URDF)
Before this commit: robot A1Z_G1Z, 13 links, 12 joints
Links:
- link camera_bracket_link: mass 0.03 -> 0.0292706516842
- link d405_link: mass 0.072 -> 0.06
